File: PWMGenerator-BrodyLaxton/PWMGenerator-BrodyLaxton.kicad_sch (KiCad schematic)
At the start: 0 parts

Commit message: iuyt
[-098
Parts:
- added C1: 0.1uF, symbol Device:C_Polarized_Small_US
- added C3: 220uF, symbol Device:C_Polarized_Small_US
- added C4: 10uF, symbol Device:C_Polarized_Small_US
- added D1, D2, D3, D4, D5: 1N4005, Diode_THT:D_DO-41_SOD81_P10.16mm_Horizontal, symbol Diode:1N4005
- added D6: LED, symbol Device:LED
- added J1: Conn_01x03_Pin, symbol Connector:Conn_01x03_Pin
- added Q1, Q2: 2N3904, Package_TO_SOT_THT:TO-92_Inline, symbol Transistor_BJT:2N3904
- added Q3, Q4: 2N3906, Package_TO_SOT_THT:TO-92_Inline, symbol Transistor_BJT:2N3906
- added R1, R10, R8: 2.2k, symbol Device:R_Small_US
- added R11: 180, symbol Device:R_Small_US
- added R2: 1M, symbol Device:R_Small_US
- added R3: 330, symbol Device:R_Small_US
- added R4: 10k, symbol Device:R_Small_US
- added R5: 220k, symbol Device:R_Small_US
- added R6: 390k, symbol Device:R_Small_US
- added R7: 22k, symbol Device:R_Small_US
- added R9: 5k, symbol Device:R_Potentiometer_US
- added SW2: SW_SPST, symbol Switch:SW_SPST
- added U1: LM339, symbol Comparator:LM339
- added U2: LM7805_TO220, Package_TO_SOT_THT:TO-220-3_Vertical, symbol Regulator_Linear:LM7805_TO220
Connections:
- new net: C4.1, J1.1 (Pin_1), Q4.3 (C), R3.1, R4.1, R5.2, R7.1, R8.1, U2.3 (VO)
- new net: R8.2, R9.1, U1.5 (+)
- new net: D6.2 (A), R3.2
- new net: D1.1 (K), D4.2 (A), SW2.2 (B)
- new net: Q4.1 (E), R11.1
- new net: C1.1, Q2.3 (C), Q3.1 (E), U1.4 (-)
- new net: D3.1 (K), D4.1 (K), D5.2 (A), R1.1, R2.1
- new net: Q1.2 (B), R2.2
- new net: Q3.2 (B), R5.1, R6.1
- new net: Q3.3 (C), R7.2
- new net: C3.1, D5.1 (K), U2.1 (VI)
- new net: Q1.3 (C), Q2.2 (B), R4.2
- new net: R10.1, U1.2
- new net: Q4.2 (B), R10.2
- new net: D2.1 (K), D3.2 (A), SW2.1 (A)
- new net GND: C1.2, C3.2, C4.2, D1.2 (A), D2.2 (A), D6.1 (K), J1.3 (Pin_3), Q1.1 (E), Q2.1 (E), R1.2, R11.2, R6.2, R9.2, R9.3, U2.2 (GND)

Commit message: 4
09
Connections:
- net VCC: now reaches C4.1, J1.1 (Pin_1), Q4.3 (C), R3.1, R4.1, R5.2, R7.1, R8.1, U2.3 (VO)
- net at Q4.1 (E), R11.1: now also J1.2 (Pin_2)
- net GNDPWR: now reaches D2.1 (K), D3.2 (A)
- net GNDPWR: no longer SW2.1 (A)
- net GND renamed GNDREF
- new net VAC: SW2.1 (A)
Other:
- moved on the sheet: C1, C3, C4, D1, D2, D3, D4, D6, Q1, Q2, Q3, Q4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

Commit message: project b b part1
xdbg
Parts:
- added F1: Polyfuse, symbol Device:Polyfuse
- added V1: VSIN, symbol Simulation_SPICE:VSIN
- C3: renamed from C1; footprint (none) -> Capacitor_SMD:C_0805_2012Metric_Pad1.18x1.45mm_HandSolder
- D1, D2, D3, D4, D5: footprint Diode_THT:D_DO-41_SOD81_P10.16mm_Horizontal -> Diode_SMD:D_0805_2012Metric_Pad1.15x1.40mm_HandSolder
- D6: value LED -> _GREEN; footprint (none) -> LED_THT:LED_D5.0mm
- J1: footprint (none) -> Connector_PinHeader_2.54mm:PinHeader_1x03_P2.54mm_Horizontal
- Q1, Q2, Q3, Q4: footprint Package_TO_SOT_THT:TO-92_Inline -> Package_TO_SOT_SMD:SOT-23
- R1, R10, R2, R3, R4, R5, R6, R7, R8: footprint (none) -> Resistor_SMD:R_0805_2012Metric
- U1: footprint (none) -> Package_SO:SOIC-14_3.9x8.7mm_P1.27mm
- renumbered C3 to C1, C4 to C2
Connections:
- net GNDPWR: now also V1.2
- net VAC: now also V1.1
- net at D1.1 (K), D4.2 (A): now also F1.2; no longer SW2.2 (B)
- new net: F1.1, SW2.2 (B)
