File: PWMGenerator-BrodyLaxton/_autosave-PWMGenerator-BrodyLaxton.kicad_sch (KiCad schematic)
At the start: 30 parts, among them J1 Conn_01x03_Pin, Q1 2N3904, Q2 2N3904, Q3 2N3906, Q4 2N3906, SW2 SW_SPST, U1 LM339, U2 LM7805_TO220

Commit message: projectb part 3
finsihed
Parts:
- added unit 4 of U1
- added unit 2 of U1
- added unit 3 of U1
- added U3: LM339, Package_SO:SOIC-14_3.9x8.7mm_P1.27mm, symbol Comparator:LM339
Connections:
- net GNDREF: now also U3.12 (V-)
- net VCC: now also U3.3 (V+)
- no-connect marks 0 -> 9
