File: PWMGenerator-BrodyLaxton/PWMGenerator-BrodyLaxton.kicad_pcb (KiCad board)
At the start: 2 copper layers, 30 parts, among them J1 Conn_01x03_Pin, Q1 2N3904, Q2 2N3904, Q3 2N3906, Q4 2N3906, SW2 SW_SPST, U1 LM339, U2 LM7805_TO220

Commit message: part 4
part 4 complete
Parts:
- removed V1: VSIN, Connector_BarrelJack:BarrelJack_SwitchcraftConxall_RAPC10U_Horizontal
- added J2: Barrel_Jack_MountingPin, Connector_BarrelJack:BarrelJack_Wuerth_694106106102_2.0x5.5mm, F.Cu at (79.2, 103.3)
- moved U1 111.4 mm to (187.5, 93.2)
- moved C2 106.7 mm to (151.7, 85.3)
- moved C1 81.8 mm to (136.0, 86.4)
- moved R9 61.7 mm to (186.1, 113.1)
- moved R10 57.4 mm to (178.2, 92.2), turned to 180 degrees
- moved C3 56.6 mm to (168.4, 117.1), turned to -90 degrees
- moved R8 52.3 mm to (174.1, 104.1)
- moved U2 52.0 mm to (155.4, 65.1)
- moved D6 49.5 mm to (96.0, 78.7), turned to 180 degrees
- moved R2 49.2 mm to (96.8, 120.3)
- moved R4 48.9 mm to (128.8, 96.8), turned to 180 degrees
- moved D5 48.3 mm to (123.7, 65.1)
- moved R6 46.9 mm to (151.6, 119.4)
- moved R11 43.2 mm to (170.9, 88.6), turned to 180 degrees
- moved Q4 41.8 mm to (169.7, 97.0)
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Routing:
- net GNDREF: track 0.00 -> 322.0 mm, vias 0 -> 9
- net VCC: track 0.00 -> 143.8 mm
- net Net-(Q2-C): track 0.00 -> 87.2 mm
- net Net-(D3-K): track 0.00 -> 71.2 mm
- net Net-(D5-K): track 0.00 -> 62.7 mm
- net VAC: track 0.00 -> 50.9 mm
- net Net-(D1-K): track 0.00 -> 46.8 mm
- net GNDPWR: track 0.00 -> 41.9 mm
- net Net-(J1-Pin_2): track 0.00 -> 32.6 mm
- net Net-(SW2-B): track 0.00 -> 30.7 mm
- net Net-(Q1-C): track 0.00 -> 29.9 mm
- net Net-(U1A-+): track 0.00 -> 28.8 mm
- net Net-(Q3-B): track 0.00 -> 24.9 mm
- net Net-(Q1-B): track 0.00 -> 20.4 mm
- net Net-(Q3-C): track 0.00 -> 16.3 mm
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- added copper zone on B.Cu, net GNDREF
- added copper zone on F.Cu, net VCC
Other:
- board outline added: 124.5 x 63.5 mm
